Commit message: add front_camera_optical_frame to fix visodom TF lookup
Co-Authored-By: Claude Sonnet 4.6 <noreply@anthropic.com>

File: urdf/front_depth.xacro (robot description, xacro)
@@ -37,4 +37,10 @@
             </xacro:inertial_box>
         </link>
+        <joint name="front_camera_optical_joint" type="fixed">
+            <parent link="front_camera_link"/>
+            <child link="front_camera_optical_frame"/>
+            <origin xyz="0 0 0" rpy="${-PI/2} 0 ${-PI/2}"/>
+        </joint>
+        <link name="front_camera_optical_frame"/>
         <gazebo reference="front_camera_link">
             <sensor name="front_d455" type="rgbd_camera">
