Commit message: Add missing back_camera_optical_frame, fix gz_frame_id for both cameras
back_depth.xacro was missing the REP-103 optical-convention frame that
front_depth.xacro already had, so back_camera had no optical frame in TF at
all. Added the same fixed local rotation front_camera's own joint uses
(independent of how the link itself is mounted). Both cameras' gazebo sensor
now reference their own optical frame instead of the mechanical link frame.

Co-Authored-By: Claude Sonnet 5 <noreply@anthropic.com>

File: urdf/back_depth.xacro (robot description, xacro)
@@ -37,7 +37,21 @@
             </xacro:inertial_box>
         </link>
+        <!-- Was missing entirely (unlike front_depth.xacro's equivalent
+             front_camera_optical_frame): without this, back_camera has no
+             REP-103 optical-convention frame in TF at all, only the
+             mechanical back_camera_link. Same fixed local rotation as
+             front's — it converts this link's own mechanical axes to
+             optical convention (x-right/y-down/z-forward), which doesn't
+             depend on how the link itself is mounted on the robot (that's
+             base2back_camera's rpy, already ${PI} to face backward). -->
+        <joint name="back_camera_optical_joint" type="fixed">
+            <parent link="back_camera_link"/>
+            <child link="back_camera_optical_frame"/>
+            <origin xyz="0 0 0" rpy="${-PI/2} 0 ${-PI/2}"/>
+        </joint>
+        <link name="back_camera_optical_frame"/>
         <gazebo reference="back_camera_link">
             <sensor name="back_d455" type="rgbd_camera">
-                <gz_frame_id>back_camera_link</gz_frame_id>
+                <gz_frame_id>back_camera_optical_frame</gz_frame_id>
                 <always_on>true</always_on>
                 <update_rate>30</update_rate>

File: urdf/front_depth.xacro (robot description, xacro)
@@ -45,5 +45,5 @@
         <gazebo reference="front_camera_link">
             <sensor name="front_d455" type="rgbd_camera">
-                <gz_frame_id>front_camera_link</gz_frame_id>
+                <gz_frame_id>front_camera_optical_frame</gz_frame_id>
                 <always_on>true</always_on>
                 <update_rate>30</update_rate>
